Commit message: telop twist with joy ps3 controlller added and working

File: description/robot.urdf.xacro (robot description, xacro)
@@ -2,5 +2,6 @@
 <robot xmlns:xacro="http://www.ros.org/wiki/xacro"  name="robot">
     <xacro:include filename="robotCore.xacro" />
-    <xacro:include filename="gazebo_control.xacro" />
+    <!-- <xacro:include filename="gazebo_control.xacro" /> -->
+    <xacro:include filename="ros2_control.xacro" />
     <xacro:include filename = "lidar.xacro" />
     <xacro:include filename = "camera.xacro" />

File: description/robotCore.xacro (robot description, xacro)
@@ -20,8 +20,14 @@
         <color rgba="0.396 0.990 0.436 1"/>
     </material>
+    <!--base_link is the root link of the robot-->
     <link name="base_link">
     </link>
+    <!--Foot print link-->
+    <jooint name="base_footprint_joint" type="fixed">
+        <origin xyz="0 0 0" rpy="0 0 0"/>
+        <parent link="base_link"/>
+        <child link="base_footprint"/>
     <joint name="chassis_joint" type="fixed">
-        <origin xyz="-0.1 0 0" rpy="0 0 0"/>
+        <origin xyz="-0.15 0 0" rpy="0 0 0"/>
         <parent link="base_link"/>
         <child link="chassis"/>
@@ -65,5 +71,5 @@
             <origin xyz="0 0 0" rpy="0 0 0"/>
             <geometry>
-                <cylinder radius="0.05" length="0.04"/>
+                <sphere radius="0.05"/>
             </geometry>
             <material name="red"/>
@@ -93,5 +99,5 @@
             <origin xyz="0 0 0" rpy="0 0 0"/>
             <geometry>
-                <cylinder radius="0.05" length="0.04"/>
+                <sphere radius="0.05"/>
             </geometry>
             <material name="green"/>
@@ -105,7 +111,7 @@
     </gazebo>
     <joint name="caster_wheel_joint" type="fixed">
-        <parent link="chassis"/>
+        <parent link="base_link"/>
         <child link="caster_wheel"/>
-        <origin xyz="0.24 0 0" rpy="0 0 0"/>
+        <origin xyz="0.15 0 0" rpy="0 0 0"/>
     </joint>
     <link name="caster_wheel">
@@ -131,3 +137,30 @@
         <mu2 value="0.001"/>
     </gazebo>
+    <joint name="caster_wheel_joint2" type="fixed">
+        <parent link="base_link"/>
+        <child link="caster_wheel2"/>
+        <origin xyz="-0.15 0 0" rpy="0 0 0"/>
+    </joint>
+        <link name="caster_wheel2">
+        <visual>
+            <geometry>
+                <sphere radius="0.05" />
+            </geometry>
+            <material name="black"/>
+        </visual>
+        <collision>
+            <geometry>
+                <sphere radius="0.05" />
+            </geometry>
+            <material name="black"/>
+        </collision>
+        <xacro:inertial_sphere mass="0.1" radius="0.05">
+            <origin xyz="0 0 0" rpy="0 0 0"/>
+        </xacro:inertial_sphere>
+    </link>
+    <gazebo reference="caster_wheel2">
+        <material>Gazebo/Black</material>
+        <mu1 value="0.001"/>
+        <mu2 value="0.001"/>
+    </gazebo>
 </robot>

Commit message: working SLAM and NAV2

File: description/robot.urdf.xacro (robot description, xacro)
@@ -1,7 +1,12 @@
 <?xml version="1.0"?>
 <robot xmlns:xacro="http://www.ros.org/wiki/xacro"  name="robot">
+    <xacro:arg name="use_ros2_control" default="true"/>
     <xacro:include filename="robotCore.xacro" />
-    <!-- <xacro:include filename="gazebo_control.xacro" /> -->
-    <xacro:include filename="ros2_control.xacro" />
+    <xacro:if value="$(arg use_ros2_control)">
+        <xacro:include filename="ros2_control.xacro" />
+    </xacro:if>
+    <xacro:unless value="$(arg use_ros2_control)">
+        <xacro:include filename="gazebo_control.xacro" />
+    </xacro:unless>
     <xacro:include filename = "lidar.xacro" />
     <xacro:include filename = "camera.xacro" />

File: description/robotCore.xacro (robot description, xacro)
@@ -24,8 +24,11 @@
     </link>
     <!--Foot print link-->
-    <jooint name="base_footprint_joint" type="fixed">
-        <origin xyz="0 0 0" rpy="0 0 0"/>
+    <joint name="base_footprint_joint" type="fixed">
         <parent link="base_link"/>
         <child link="base_footprint"/>
+        <origin xyz="0 0 0" rpy="0 0 0"/>
+    </joint>
+    <link name="base_footprint">
+    </link>
     <joint name="chassis_joint" type="fixed">
         <origin xyz="-0.15 0 0" rpy="0 0 0"/>
